Commit message: fix relatice paths in urdf

File: src/so101_description/urdf/so101_new_calib.urdf (robot description, URDF)
Before this commit: robot so101_new_calib, 8 links, 7 joints
Links:
- link base_link: geometry collision mesh filename=package://so101_description/meshesbase_motor_holder_so101_v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; collision mesh filename=package://so101_description/meshesbase_so101_v2.stl
- link gripper_link: geometry collision mesh filename=package://so101_description/meshessts3215_03a_v1.stl; collision mesh filename=package://so101_description/mesheswrist_roll_follower_so101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
- link lower_arm_link: geometry collision mesh filename=package://so101_description/meshesmotor_holder_so101_wrist_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; collision mesh filename=package://so101_description/meshessts3215_03a_v1.stl
- link moving_jaw_so101_v1_link: geometry collision mesh filename=package://so101_description/meshesmoving_jaw_so101_v1.stl; visual mesh filename=package://so101_description/meshesmoving_jaw_so101_v1.stl
- link shoulder_link: geometry collision mesh filename=package://so101_description/meshesmotor_holder_so101_base_v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; collision mesh filename=package://so101_description/meshesrotation_pitch_so101_v1.s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
- link upper_arm_link: geometry collision mesh filename=package://so101_description/meshessts3215_03a_v1.stl; collision mesh filename=package://so101_description/meshesupper_arm_so101_v1.stl
- link wrist_link: geometry collision mesh filename=package://so101_description/meshessts3215_03a_no_horn_v1.stl; collision mesh filename=package://so101_description/mesheswrist_roll_pitch_so101_v2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
