Commit message: add urdf with camera

File: src/so101_description/urdf/so101_new_calib_camera.urdf (robot description, URDF)
Before this commit: robot so101_new_calib, 8 links, 7 joints
Links:
- added link wrist_camera_link, mass 0.015; collision mesh filename=package://so101_description/meshes/wrist_camera_so101_v1.stl; visual mesh filename=package://so101_description/meshes/wrist_camera_so101_v1.stl
- added link wrist_camera_mount_link, mass 0.02; collision mesh filename=package://so101_description/meshes/wrist_camera_mount_so101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 scale=0.001 0.001 0.001; visual mesh filename=package://so101_description/meshes/wrist_camera_mount_so101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 scale=0.001 0.001 0.001
Joints:
- added joint wrist_camera_joint: type fixed, parent wrist_camera_mount_link, child wrist_camera_link, origin xyz=-0.04941 -0.03813 0.0175 rpy=0 -1.5708 -2.0076
- added joint wrist_camera_mount_joint: type fixed, parent gripper_link, child wrist_camera_mount_link, origin xyz=-0.0150 0.0240 -0.0315 rpy=-1.5708 -0.0008 -1.5708
