Commit message: convert urdf to xacro

File: src/so101_description/urdf/so101.urdf.xacro (robot description, xacro)
@@ -2,5 +2,7 @@
 <!-- Generated using onshape-to-robot -->
 <!-- Onshape https://cad.onshape.com/documents/7715cc284bb430fe6dab4ffd/w/4fd0791b683777b02f8d975a/e/826c553ede3b7592eb9ca800 -->
-<robot name="so101_new_calib">
+<!-- Derived from so101_new_calib.urdf: adds wrist camera mount + wrist camera (Hex-Nut 32x32 UVC module form factor) -->
+<robot name="so101_new_calib_camera" xmlns:xacro="http://www.ros.org/wiki/xacro">
+<xacro:arg name="use_camera" default="true"/>
   <!-- Materials -->
   <material name="3d_printed">
@@ -327,14 +329,4 @@
     <limit effort="10" velocity="10" lower="-0.174533" upper="1.74533"/>
   </joint>
-  <transmission name="gripper_trans">
-    <type>transmission_interface/SimpleTransmission</type>
-    <joint name="gripper">
-      <hardwareInterface>hardware_interface/PositionJointInterface</hardwareInterface>
-    </joint>
-    <actuator name="motor6">
-      <hardwareInterface>hardware_interface/PositionJointInterface</hardwareInterface>
-      <mechanicalReduction>1</mechanicalReduction>
-    </actuator>
-  </transmission>
   <!-- Joint from wrist to gripper -->
   <joint name="wrist_roll" type="revolute">
@@ -345,14 +337,4 @@
     <limit effort="10" velocity="10" lower="-2.74385" upper="2.84121"/>
   </joint>
-  <transmission name="wrist_roll_trans">
-    <type>transmission_interface/SimpleTransmission</type>
-    <joint name="wrist_roll">
-      <hardwareInterface>hardware_interface/PositionJointInterface</hardwareInterface>
-    </joint>
-    <actuator name="motor5">
-      <hardwareInterface>hardware_interface/PositionJointInterface</hardwareInterface>
-      <mechanicalReduction>1</mechanicalReduction>
-    </actuator>
-  </transmission>
   <!-- Joint from lower_arm to wrist -->
   <joint name="wrist_flex" type="revolute">
@@ -363,14 +345,4 @@
     <limit effort="10" velocity="10" lower="-1.65806" upper="1.65806"/>
   </joint>
-  <transmission name="wrist_flex_trans">
-    <type>transmission_interface/SimpleTransmission</type>
-    <joint name="wrist_flex">
-      <hardwareInterface>hardware_interface/PositionJointInterface</hardwareInterface>
-    </joint>
-    <actuator name="motor4">
-      <hardwareInterface>hardware_interface/PositionJointInterface</hardwareInterface>
-      <mechanicalReduction>1</mechanicalReduction>
-    </actuator>
-  </transmission>
   <!-- Joint from upper_arm to lower_arm -->
   <!-- Note: 5-degree calibration offset applied to joint limits -->
@@ -382,14 +354,4 @@
     <limit effort="10" velocity="10" lower="-1.69" upper="1.69"/>
   </joint>
-  <transmission name="elbow_flex_trans">
-    <type>transmission_interface/SimpleTransmission</type>
-    <joint name="elbow_flex">
-      <hardwareInterface>hardware_interface/PositionJointInterface</hardwareInterface>
-    </joint>
-    <actuator name="motor3">
-      <hardwareInterface>hardware_interface/PositionJointInterface</hardwareInterface>
-      <mechanicalReduction>1</mechanicalReduction>
-    </actuator>
-  </transmission>
   <!-- Joint from shoulder to upper_arm -->
   <joint name="shoulder_lift" type="revolute">
@@ -400,14 +362,4 @@
     <limit effort="10" velocity="10" lower="-1.74533" upper="1.74533"/>
   </joint>
-  <transmission name="shoulder_lift_trans">
-    <type>transmission_interface/SimpleTransmission</type>
-    <joint name="shoulder_lift">
-      <hardwareInterface>hardware_interface/PositionJointInterface</hardwareInterface>
-    </joint>
-    <actuator name="motor2">
-      <hardwareInterface>hardware_interface/PositionJointInterface</hardwareInterface>
-      <mechanicalReduction>1</mechanicalReduction>
-    </actuator>
-  </transmission>
   <!-- Joint from base to shoulder -->
   <joint name="shoulder_pan" type="revolute">
@@ -418,13 +370,61 @@
     <limit effort="10" velocity="10" lower="-1.91986" upper="1.91986"/>
   </joint>
-  <transmission name="shoulder_pan_trans">
-    <type>transmission_interface/SimpleTransmission</type>
-    <joint name="shoulder_pan">
-      <hardwareInterface>hardware_interface/PositionJointInterface</hardwareInterface>
-    </joint>
-    <actuator name="motor1">
-      <hardwareInterface>hardware_interface/PositionJointInterface</hardwareInterface>
-      <mechanicalReduction>1</mechanicalReduction>
-    </actuator>
-  </transmission>
+  <!-- Link wrist_camera_mount -->
+  <xacro:if value="$(arg use_camera)">
+  <link name="wrist_camera_mount_link">
+    <inertial>
+      <origin xyz="0 0 0" rpy="0 0 0"/>
+      <mass value="0.02"/>
+      <inertia ixx="1e-5" ixy="0" ixz="0" iyy="1e-5" iyz="0" izz="1e-5"/>
+    </inertial>
+    <!-- Part wrist_camera_mount_so101_v1 (Hex-Nut Recess, 32x32 UVC module form factor) -->
+    <visual>
+      <origin xyz="0 0 0" rpy="0 0 0"/>
+      <geometry>
+        <mesh filename="package://so101_description/meshes/wrist_camera_mount_so101_v1.stl" scale="0.001 0.001 0.001"/>
+      </geometry>
+      <material name="3d_printed"/>
+    </visual>
+    <collision>
+      <origin xyz="0 0 0" rpy="0 0 0"/>
+      <geometry>
+        <mesh filename="package://so101_description/meshes/wrist_camera_mount_so101_v1.stl" scale="0.001 0.001 0.001"/>
+      </geometry>
+    </collision>
+  </link>
+  <!-- Link wrist_camera -->
+  <link name="wrist_camera_link">
+    <inertial>
+      <origin xyz="0 0 0" rpy="0 0 0"/>
+      <mass value="0.015"/>
+      <inertia ixx="1e-5" ixy="0" ixz="0" iyy="1e-5" iyz="0" izz="1e-5"/>
+    </inertial>
+    <!-- Part wrist_camera_so101_v1 -->
+    <visual>
+      <origin xyz="0 0 0" rpy="0 0 0"/>
+      <geometry>
+        <mesh filename="package://so101_description/meshes/wrist_camera_so101_v1.stl"/>
+      </geometry>
+      <material name="sts3215"/>
+    </visual>
+    <collision>
+      <origin xyz="0 0 0" rpy="0 0 0"/>
+      <geometry>
+        <mesh filename="package://so101_description/meshes/wrist_camera_so101_v1.stl"/>
+      </geometry>
+    </collision>
+  </link>
+  <!-- Joint from gripper to wrist_camera_mount -->
+  <joint name="wrist_camera_mount_joint" type="fixed">
+    <origin xyz="-0.0150 0.0240 -0.0315" rpy="-1.5708 -0.0008 -1.5708"/>
+    <parent link="gripper_link"/>
+    <child link="wrist_camera_mount_link"/>
+  </joint>
+  <!-- Joint from wrist_camera_mount to wrist_camera -->
+  <joint name="wrist_camera_joint" type="fixed">
+    <origin xyz="-0.04941 -0.03813 0.0175" rpy="0 -1.5708 -2.0076"/>
+    <parent link="wrist_camera_mount_link"/>
+    <child link="wrist_camera_link"/>
+  </joint>
+  </xacro:if>
 </robot>

Commit message: add control packages for arm

File: src/so101_description/urdf/so101.urdf.xacro (robot description, xacro)
@@ -428,3 +428,21 @@
   </joint>
   </xacro:if>
+<xacro:macro name="joint_interfaces" params="name">
+  <joint name="${name}">
+    <command_interface name="position"/>
+    <state_interface name="position"/>
+    <state_interface name="velocity"/>
+  </joint>
+</xacro:macro>
+<ros2_control name="so101_system" type="system">
+  <hardware>
+    <plugin>mock_components/GenericSystem</plugin>
+  </hardware>
+  <xacro:joint_interfaces name="shoulder_pan"/>
+  <xacro:joint_interfaces name="shoulder_lift"/>
+  <xacro:joint_interfaces name="elbow_flex"/>
+  <xacro:joint_interfaces name="wrist_flex"/>
+  <xacro:joint_interfaces name="wrist_roll"/>
+  <xacro:joint_interfaces name="gripper"/>
+</ros2_control>
 </robot>
